Commit message: Update imu.urdf.xacro
updated IMU position to new orientation

File: urdf/sensors/imu.urdf.xacro (robot description, xacro)
@@ -5,5 +5,5 @@
       <parent link="base_link"/>
       <child link="imu_link"/>
-      <origin xyz="0.01 0 .0916" rpy="0 1.57 0"/>
+      <origin xyz="0.01 0 .0762" rpy="0 0 0"/>
     </joint>
   </xacro:macro>

Commit message: updated for wood stake

File: urdf/sensors/imu.urdf.xacro (robot description, xacro)
@@ -5,5 +5,5 @@
       <parent link="base_link"/>
       <child link="imu_link"/>
-      <origin xyz="0.01 0 .0762" rpy="0 0 0"/>
+      <origin xyz="0 0 .2032" rpy="0 0 0"/>
     </joint>
   </xacro:macro>

Commit message: Update imu.urdf.xacro

File: urdf/sensors/imu.urdf.xacro (robot description, xacro)
@@ -5,5 +5,5 @@
       <parent link="base_link"/>
       <child link="imu_link"/>
-      <origin xyz="0 0 .2032" rpy="0 0 0"/>
+      <origin xyz="0 0 .2032" rpy="-0.174533 -0.10472 0"/>
     </joint>
   </xacro:macro>
